File: KiCAD/8-Bit CPU/Clock_AVR.sch (KiCad schematic (older format))
At the start: 5 parts, among them J6 AVRISP, U53 ATtiny45-20SU

Commit message: KiCAD files update & Gerbers
Parts:
- U53: footprint Package_SO:SOIC-8_3.9x4.9mm_P1.27mm -> Package_SO:SOIC-8_5.275x5.275mm_P1.27mm
- renumbered RN31 to RN33
Changed lines of the file:
@@
 $Descr A4 11693 8268
 encoding utf-8
-Sheet 30 29
+Sheet 29 29
 Title ""
 Date ""
-Rev ""
+Rev "C"
 Comp ""
 Comment1 ""
@@
 F 0 "U53" H 4471 3646 50  0000 R CNN
 F 1 "ATtiny45-20SU" H 4471 3555 50  0000 R CNN
-F 2 "Package_SO:SOIC-8_3.9x4.9mm_P1.27mm" H 5000 3600 50  0001 C CIN
+F 2 "Package_SO:SOIC-8_5.275x5.275mm_P1.27mm" H 5000 3600 50  0001 C CIN
 F 3 "http://ww1.microchip.com/downloads/en/DeviceDoc/atmel-2586-avr-8-bit-microcontroller-attiny25-attiny45-attiny85_datasheet.pdf" H 5000 3600 50  0001 C CNN
 	1    5000 3600
@@
 CLK
 $Comp
-L power:VCC #PWR0292
+L power:VCC #PWR0289
 U 1 1 5D714B96
 P 5000 3000
-F 0 "#PWR0292" H 5000 2850 50  0001 C CNN
+F 0 "#PWR0289" H 5000 2850 50  0001 C CNN
 F 1 "VCC" H 5017 3173 50  0000 C CNN
 F 2 "" H 5000 3000 50  0001 C CNN
@@
 $EndComp
 $Comp
-L power:GND #PWR0293
+L power:GND #PWR0296
 U 1 1 5D71501A
 P 5000 4200
-F 0 "#PWR0293" H 5000 3950 50  0001 C CNN
+F 0 "#PWR0296" H 5000 3950 50  0001 C CNN
 F 1 "GND" H 5005 4027 50  0000 C CNN
 F 2 "" H 5000 4200 50  0001 C CNN
@@
 AR Path="/5D643828/5D4645A0/5D717CBF" Ref="#PWR?"  Part="1"
 AR Path="/5D5F87DE/5D717CBF" Ref="#PWR?"  Part="1"
-AR Path="/5D5F87DE/5D6FC11A/5D717CBF" Ref="#PWR0295"  Part="1"
-F 0 "#PWR0295" H 5850 4150 50  0001 C CNN
+AR Path="/5D5F87DE/5D6FC11A/5D717CBF" Ref="#PWR0298"  Part="1"
+F 0 "#PWR0298" H 5850 4150 50  0001 C CNN
 F 1 "GND" H 5855 4227 50  0000 C CNN
 F 2 "" H 5850 4400 50  0001 C CNN
@@
 P 5850 4100
 AR Path="/5D5F87DE/5D717CC5" Ref="#PWR?"  Part="1"
-AR Path="/5D5F87DE/5D6FC11A/5D717CC5" Ref="#PWR0294"  Part="1"
-F 0 "#PWR0294" H 5850 3950 50  0001 C CNN
+AR Path="/5D5F87DE/5D6FC11A/5D717CC5" Ref="#PWR0295"  Part="1"
+F 0 "#PWR0295" H 5850 3950 50  0001 C CNN
 F 1 "VCC" H 5867 4273 50  0000 C CNN
 F 2 "" H 5850 4100 50  0001 C CNN
@@
 AR Path="/5D5DCCF9/5D71DF6A" Ref="#PWR?"  Part="1"
 AR Path="/5D5C9807/5D71DF6A" Ref="#PWR?"  Part="1"
-AR Path="/5D5F87DE/5D6FC11A/5D71DF6A" Ref="#PWR0298"  Part="1"
-F 0 "#PWR0298" H 6650 4100 50  0001 C CNN
+AR Path="/5D5F87DE/5D6FC11A/5D71DF6A" Ref="#PWR0297"  Part="1"
+F 0 "#PWR0297" H 6650 4100 50  0001 C CNN
 F 1 "GND" H 6655 4177 50  0000 C CNN
 F 2 "" H 6650 4350 50  0001 C CNN
@@
 AR Path="/5D5DCCF9/5D71DF75" Ref="#PWR?"  Part="1"
 AR Path="/5D5C9807/5D71DF75" Ref="#PWR?"  Part="1"
-AR Path="/5D5F87DE/5D6FC11A/5D71DF75" Ref="#PWR0300"  Part="1"
-F 0 "#PWR0300" H 6750 3750 50  0001 C CNN
+AR Path="/5D5F87DE/5D6FC11A/5D71DF75" Ref="#PWR0294"  Part="1"
+F 0 "#PWR0294" H 6750 3750 50  0001 C CNN
 F 1 "VCC" V 6750 4000 50  0000 L CNN
 F 2 "" H 6750 3900 50  0001 C CNN
@@
 AR Path="/5D613953/5D5E5DC0/5D754D36" Ref="RN?"  Part="1"
 AR Path="/5D5EAD14/5D754D36" Ref="RN?"  Part="1"
-AR Path="/5D5F87DE/5D6FC11A/5D754D36" Ref="RN31"  Part="1"
-F 0 "RN31" V 6533 3300 50  0000 C CNN
+AR Path="/5D5F87DE/5D6FC11A/5D754D36" Ref="RN33"  Part="1"
+F 0 "RN33" V 6533 3300 50  0000 C CNN
 F 1 "10k" V 6624 3300 50  0000 C CNN
 F 2 "Resistor_SMD:R_Array_Concave_4x0603" V 7225 3300 50  0001 C CNN
@@
 	5600 3400 5850 3400
 $Comp
-L power:VCC #PWR0301
+L power:VCC #PWR0290
 U 1 1 5D75664A
 P 7150 3100
-F 0 "#PWR0301" H 7150 2950 50  0001 C CNN
+F 0 "#PWR0290" H 7150 2950 50  0001 C CNN
 F 1 "VCC" V 7167 3228 50  0000 L CNN
 F 2 "" H 7150 3100 50  0001 C CNN
@@
 	7350 3400 7150 3400
 $Comp
-L power:VCC #PWR0299
+L power:VCC #PWR0291
 U 1 1 5D755BBC
 P 6750 3200
-F 0 "#PWR0299" H 6750 3050 50  0001 C CNN
+F 0 "#PWR0291" H 6750 3050 50  0001 C CNN
 F 1 "VCC" V 6768 3327 50  0000 L CNN
 F 2 "" H 6750 3200 50  0001 C CNN
@@
 AR Path="/5D5DCCF9/5D760959" Ref="#PWR?"  Part="1"
 AR Path="/5D5C9807/5D760959" Ref="#PWR?"  Part="1"
-AR Path="/5D5F87DE/5D6FC11A/5D760959" Ref="#PWR0297"  Part="1"
-F 0 "#PWR0297" H 6250 3600 50  0001 C CNN
+AR Path="/5D5F87DE/5D6FC11A/5D760959" Ref="#PWR0293"  Part="1"
+F 0 "#PWR0293" H 6250 3600 50  0001 C CNN
 F 1 "GND" H 6255 3677 50  0000 C CNN
 F 2 "" H 6250 3850 50  0001 C CNN
@@
 $EndComp
 $Comp
-L power:VCC #PWR0296
+L power:VCC #PWR0292
 U 1 1 5D760BF8
 P 6250 3350
-F 0 "#PWR0296" H 6250 3200 50  0001 C CNN
+F 0 "#PWR0292" H 6250 3200 50  0001 C CNN
 F 1 "VCC" H 6267 3523 50  0000 C CNN
 F 2 "" H 6250 3350 50  0001 C CNN
