File: KiCAD/8-Bit CPU/Control.sch (KiCad schematic (older format))
At the start: 2 parts

Commit message: KiCAD cleanup - Revision A
Revision A Known Issues:
 * ATTiny45 has incorrect footprint
 * Flags register is redundant (The ATMega16's output port is a register)
 * Power jack pinout is wrong (12V shorted to ground)
 * Step counter reset logic is wrong (Active high signalling, Active low input)
 * ALU output indicator not connected
 * HLT indicator missing
 * EEPROMs can't be page written due to addressing setup (minor annoyance)
 * Flags Logic uses NAND gates instead of AND (fixed on the board I built)
 * Programmer needs to be able to toggle EEPROM outputs and Addressing Devices
    with different signals to enable reading.
Parts:
- added U28: 74HC00, jcf:SOIC-14_3.9x8.7mm_P1.27mm_JCF, symbol 74xx:74HC00
- added U30: 74HC32, Package_SO:SOIC-14_3.9x8.7mm_P1.27mm, symbol 74xx:74LS32
Connections:
- net A0: now also U28.13
- net A1: now also U28.10
- net A2: now also U28.5
- net F1: now also U28.12
- net F2: now also U28.9
- net F3: now also U28.4
- new net: U30.11, U30.9
- new net: U28.6, U30.12
- new net: U28.8, U30.13
- new net: U28.11, U30.10
- new net Address Buffer/A12: U30.8
Other:
- note added: "These Gates should be HC08 AND\nHC00 NAND is an error."
- note added: "~OE~ should be 2 signals\nEEPROM ~OE~ and\nBUFFER ~OE"

Commit message: KiCAD files update & Gerbers
Parts:
- removed R28, R29: 10k, Resistor_SMD:R_0805_2012Metric, symbol Device:R
- removed U28: 74HC00, jcf:SOIC-14_3.9x8.7mm_P1.27mm_JCF, symbol 74xx:74HC00
- removed U30: 74HC32, Package_SO:SOIC-14_3.9x8.7mm_P1.27mm, symbol 74xx:74LS32
- added C34, C35, C36: 100n, Capacitor_SMD:C_0805_2012Metric, symbol Device:C
- added U27: 74HC08, jcf:SOIC-14_3.9x8.7mm_P1.27mm_JCF, symbol 74xx:74LS08
- added U28, U29: 74HC1G32, Package_SO:TSOP-5_1.65x3.05mm_P0.95mm, symbol jcf-digital:74HC1G32
Connections:
- net labels added: FL, ~AE, ~EE, ~MSR
- net labels removed: MSR, ~OE
- wire segments 205 -> 206
- no-connect marks 0 -> 1
Other:
- note removed: "These Gates should be HC08 AND\nHC00 NAND is an error."
- note removed: "~OE~ should be 2 signals\nEEPROM ~OE~ and\nBUFFER ~OE"
