File: KiCAD/8-Bit CPU/Control_AddrBuff.sch (KiCad schematic (older format))
At the start: 4 parts, among them U31 74HC245, U32 74HC245

Commit message: KiCAD files update & Gerbers
Parts:
- renumbered C38 to C39, C39 to C40, U31 to U32, U32 to U33
Connections:
- net A10: now also U33.16 (B2); no longer U33.4 (A2)
- net A11: now also U33.17 (B1); no longer U33.3 (A1)
- net A12: now also U33.18 (B0); no longer U33.2 (A0)
- net A8: now also U33.14 (B4); no longer U33.6 (A4)
- net A9: now also U33.15 (B3); no longer U33.5 (A3)
- net B10: now also U33.4 (A2); no longer U33.16 (B2)
- net B11: now also U33.3 (A1); no longer U33.17 (B1)
- net B12: now also U33.2 (A0); no longer U33.18 (B0)
- net B8: now also U33.6 (A4); no longer U33.14 (B4)
- net B9: now also U33.5 (A3); no longer U33.15 (B3)
- net GND: now also U33.1 (A->B), U33.11 (B7), U33.12 (B6), U33.13 (B5); no longer U33.7 (A5), U33.8 (A6), U33.9 (A7)
- net VCC: no longer U33.1 (A->B)
Other:
- moved on the sheet: C40
Changed lines of the file:
@@
 $Descr A4 11693 8268
 encoding utf-8
-Sheet 26 29
+Sheet 21 29
 Title ""
 Date ""
-Rev ""
+Rev "C"
 Comp ""
 Comment1 ""
@@
 AR Path="/5D50DAD7/5D510BA9" Ref="U?"  Part="1"
 AR Path="/5D59955E/5D510BA9" Ref="U?"  Part="1"
-AR Path="/5D6D875D/5D50DAD7/5D510BA9" Ref="U31"  Part="1"
-F 0 "U31" H 5750 3200 50  0000 L CNN
+AR Path="/5D6D875D/5D50DAD7/5D510BA9" Ref="U32"  Part="1"
+F 0 "U32" H 5750 3200 50  0000 L CNN
 F 1 "74HC245" H 5750 3100 50  0000 L CNN
 F 2 "Package_SO:SOIC-20W_7.5x12.8mm_P1.27mm" H 5700 2400 50  0001 C CNN
@@
 AR Path="/5D50DAD7/5D510BB6" Ref="#PWR?"  Part="1"
 AR Path="/5D59955E/5D510BB6" Ref="#PWR?"  Part="1"
-AR Path="/5D6D875D/5D50DAD7/5D510BB6" Ref="#PWR0194"  Part="1"
-F 0 "#PWR0194" H 5700 2950 50  0001 C CNN
+AR Path="/5D6D875D/5D50DAD7/5D510BB6" Ref="#PWR0191"  Part="1"
+F 0 "#PWR0191" H 5700 2950 50  0001 C CNN
 F 1 "GND" H 5705 3027 50  0000 C CNN
 F 2 "" H 5700 3200 50  0001 C CNN
@@
 AR Path="/5D50DAD7/5D510BBE" Ref="#PWR?"  Part="1"
 AR Path="/5D59955E/5D510BBE" Ref="#PWR?"  Part="1"
-AR Path="/5D6D875D/5D50DAD7/5D510BBE" Ref="#PWR0193"  Part="1"
-F 0 "#PWR0193" H 5700 1450 50  0001 C CNN
+AR Path="/5D6D875D/5D50DAD7/5D510BBE" Ref="#PWR0188"  Part="1"
+F 0 "#PWR0188" H 5700 1450 50  0001 C CNN
 F 1 "VCC" H 5717 1773 50  0000 C CNN
 F 2 "" H 5700 1600 50  0001 C CNN
@@
 AR Path="/5D50DAD7/5D510BC4" Ref="#PWR?"  Part="1"
 AR Path="/5D59955E/5D510BC4" Ref="#PWR?"  Part="1"
-AR Path="/5D6D875D/5D50DAD7/5D510BC4" Ref="#PWR0191"  Part="1"
-F 0 "#PWR0191" H 5200 2650 50  0001 C CNN
+AR Path="/5D6D875D/5D50DAD7/5D510BC4" Ref="#PWR0189"  Part="1"
+F 0 "#PWR0189" H 5200 2650 50  0001 C CNN
 F 1 "VCC" V 5218 2927 50  0000 L CNN
 F 2 "" H 5200 2800 50  0001 C CNN
@@
 AR Path="/5D50DAD7/5D511952" Ref="C?"  Part="1"
 AR Path="/5D59955E/5D511952" Ref="C?"  Part="1"
-AR Path="/5D6D875D/5D50DAD7/5D511952" Ref="C38"  Part="1"
-F 0 "C38" H 6315 3096 50  0000 L CNN
+AR Path="/5D6D875D/5D50DAD7/5D511952" Ref="C39"  Part="1"
+F 0 "C39" H 6315 3096 50  0000 L CNN
 F 1 "100n" H 6315 3005 50  0000 L CNN
 F 2 "Capacitor_SMD:C_0805_2012Metric" H 6238 2900 50  0001 C CNN
@@
 AR Path="/5D50DAD7/5D511959" Ref="#PWR?"  Part="1"
 AR Path="/5D59955E/5D511959" Ref="#PWR?"  Part="1"
-AR Path="/5D6D875D/5D50DAD7/5D511959" Ref="#PWR0198"  Part="1"
-F 0 "#PWR0198" H 6200 2950 50  0001 C CNN
+AR Path="/5D6D875D/5D50DAD7/5D511959" Ref="#PWR0192"  Part="1"
+F 0 "#PWR0192" H 6200 2950 50  0001 C CNN
 F 1 "GND" H 6205 3027 50  0000 C CNN
 F 2 "" H 6200 3200 50  0001 C CNN
@@
 AR Path="/5D50DAD7/5D51195F" Ref="#PWR?"  Part="1"
 AR Path="/5D59955E/5D51195F" Ref="#PWR?"  Part="1"
-AR Path="/5D6D875D/5D50DAD7/5D51195F" Ref="#PWR0197"  Part="1"
-F 0 "#PWR0197" H 6200 2750 50  0001 C CNN
+AR Path="/5D6D875D/5D50DAD7/5D51195F" Ref="#PWR0190"  Part="1"
+F 0 "#PWR0190" H 6200 2750 50  0001 C CNN
 F 1 "VCC" H 6217 3073 50  0000 C CNN
 F 2 "" H 6200 2900 50  0001 C CNN
 F 3 "" H 6200 2900 50  0001 C CNN
 	1    6200 2900
-	1    0    0    -1
-$EndComp
-$Comp
-L 74xx:74LS245 U?
-U 1 1 5D511BC2
-P 5700 4650
-AR Path="/5D511BC2" Ref="U?"  Part="1"
-AR Path="/5D50DAD7/5D511BC2" Ref="U?"  Part="1"
-AR Path="/5D59955E/5D511BC2" Ref="U?"  Part="1"
-AR Path="/5D6D875D/5D50DAD7/5D511BC2" Ref="U32"  Part="1"
-F 0 "U32" H 5750 5450 50  0000 L CNN
-F 1 "74HC245" H 5750 5350 50  0000 L CNN
-F 2 "Package_SO:SOIC-20W_7.5x12.8mm_P1.27mm" H 5700 4650 50  0001 C CNN
-F 3 "http://www.ti.com/lit/gpn/sn74LS245" H 5700 4650 50  0001 C CNN
-	1    5700 4650
 	1    0    0    -1
 $EndComp
@@
 AR Path="/5D50DAD7/5D511BD7" Ref="#PWR?"  Part="1"
 AR Path="/5D59955E/5D511BD7" Ref="#PWR?"  Part="1"
-AR Path="/5D6D875D/5D50DAD7/5D511BD7" Ref="#PWR0195"  Part="1"
-F 0 "#PWR0195" H 5700 3700 50  0001 C CNN
+AR Path="/5D6D875D/5D50DAD7/5D511BD7" Ref="#PWR0193"  Part="1"
+F 0 "#PWR0193" H 5700 3700 50  0001 C CNN
 F 1 "VCC" H 5717 4023 50  0000 C CNN
 F 2 "" H 5700 3850 50  0001 C CNN
@@
 	1    5700 3850
 	1    0    0    -1
-$EndComp
-$Comp
-L power:VCC #PWR?
-U 1 1 5D511BDD
-P 5200 5050
-AR Path="/5D511BDD" Ref="#PWR?"  Part="1"
-AR Path="/5D50DAD7/5D511BDD" Ref="#PWR?"  Part="1"
-AR Path="/5D59955E/5D511BDD" Ref="#PWR?"  Part="1"
-AR Path="/5D6D875D/5D50DAD7/5D511BDD" Ref="#PWR0192"  Part="1"
-F 0 "#PWR0192" H 5200 4900 50  0001 C CNN
-F 1 "VCC" V 5218 5177 50  0000 L CNN
-F 2 "" H 5200 5050 50  0001 C CNN
-F 3 "" H 5200 5050 50  0001 C CNN
-	1    5200 5050
-	0    -1   -1   0
 $EndComp
 Text HLabel 5100 4550 0    50   Input ~ 0
@@
 L Device:C C?
 U 1 1 5D511BFB
-P 6200 5300
+P 6900 5300
 AR Path="/5D4EE537/5D511BFB" Ref="C?"  Part="1"
 AR Path="/5D50DAD7/5D511BFB" Ref="C?"  Part="1"
 AR Path="/5D59955E/5D511BFB" Ref="C?"  Part="1"
-AR Path="/5D6D875D/5D50DAD7/5D511BFB" Ref="C39"  Part="1"
-F 0 "C39" H 6315 5346 50  0000 L CNN
-F 1 "100n" H 6315 5255 50  0000 L CNN
-F 2 "Capacitor_SMD:C_0805_2012Metric" H 6238 5150 50  0001 C CNN
-F 3 "~" H 6200 5300 50  0001 C CNN
-	1    6200 5300
+AR Path="/5D6D875D/5D50DAD7/5D511BFB" Ref="C40"  Part="1"
+F 0 "C40" H 7015 5346 50  0000 L CNN
+F 1 "100n" H 7015 5255 50  0000 L CNN
+F 2 "Capacitor_SMD:C_0805_2012Metric" H 6938 5150 50  0001 C CNN
+F 3 "~" H 6900 5300 50  0001 C CNN
+	1    6900 5300
 	1    0    0    -1
 $EndComp
@@
 L power:GND #PWR?
 U 1 1 5D511C02
-P 6200 5450
+P 6900 5450
 AR Path="/5D511C02" Ref="#PWR?"  Part="1"
 AR Path="/5D4EE537/5D511C02" Ref="#PWR?"  Part="1"
 AR Path="/5D50DAD7/5D511C02" Ref="#PWR?"  Part="1"
 AR Path="/5D59955E/5D511C02" Ref="#PWR?"  Part="1"
-AR Path="/5D6D875D/5D50DAD7/5D511C02" Ref="#PWR0200"  Part="1"
-F 0 "#PWR0200" H 6200 5200 50  0001 C CNN
-F 1 "GND" H 6205 5277 50  0000 C CNN
-F 2 "" H 6200 5450 50  0001 C CNN
-F 3 "" H 6200 5450 50  0001 C CNN
-	1    6200 5450
+AR Path="/5D6D875D/5D50DAD7/5D511C02" Ref="#PWR0198"  Part="1"
+F 0 "#PWR0198" H 6900 5200 50  0001 C CNN
+F 1 "GND" H 6905 5277 50  0000 C CNN
+F 2 "" H 6900 5450 50  0001 C CNN
+F 3 "" H 6900 5450 50  0001 C CNN
+	1    6900 5450
 	1    0    0    -1
 $EndComp
@@
 L power:VCC #PWR?
 U 1 1 5D511C08
-P 6200 5150
+P 6900 5150
 AR Path="/5D511C08" Ref="#PWR?"  Part="1"
 AR Path="/5D4EE537/5D511C08" Ref="#PWR?"  Part="1"
 AR Path="/5D50DAD7/5D511C08" Ref="#PWR?"  Part="1"
 AR Path="/5D59955E/5D511C08" Ref="#PWR?"  Part="1"
-AR Path="/5D6D875D/5D50DAD7/5D511C08" Ref="#PWR0199"  Part="1"
-F 0 "#PWR0199" H 6200 5000 50  0001 C CNN
-F 1 "VCC" H 6217 5323 50  0000 C CNN
-F 2 "" H 6200 5150 50  0001 C CNN
-F 3 "" H 6200 5150 50  0001 C CNN
-	1    6200 5150
+AR Path="/5D6D875D/5D50DAD7/5D511C08" Ref="#PWR0195"  Part="1"
+F 0 "#PWR0195" H 6900 5000 50  0001 C CNN
+F 1 "VCC" H 6917 5323 50  0000 C CNN
+F 2 "" H 6900 5150 50  0001 C CNN
+F 3 "" H 6900 5150 50  0001 C CNN
+	1    6900 5150
 	1    0    0    -1
 $EndComp
@@
 AR Path="/5D50DAD7/5D512376" Ref="#PWR?"  Part="1"
 AR Path="/5D59955E/5D512376" Ref="#PWR?"  Part="1"
-AR Path="/5D6D875D/5D50DAD7/5D512376" Ref="#PWR0190"  Part="1"
-F 0 "#PWR0190" H 5100 4650 50  0001 C CNN
+AR Path="/5D6D875D/5D50DAD7/5D512376" Ref="#PWR0194"  Part="1"
+F 0 "#PWR0194" H 5100 4650 50  0001 C CNN
 F 1 "GND" H 4950 4850 50  0000 C CNN
 F 2 "" H 5100 4900 50  0001 C CNN
@@
 Wire Wire Line
 	5100 4850 5100 4750
-Wire Wire Line
-	5200 5150 4800 5150
-Wire Wire Line
-	4800 5150 4800 2900
-Wire Wire Line
-	4800 2900 5200 2900
 Text HLabel 4700 2900 0    50   Input ~ 0
 ~OE
-Wire Wire Line
-	4700 2900 4800 2900
-Connection ~ 4800 2900
 NoConn ~ 6200 4650
 NoConn ~ 6200 4750
 NoConn ~ 6200 4850
+$Comp
+L 74xx:74LS245 U?
+U 1 1 5D511BC2
+P 5700 4650
+AR Path="/5D511BC2" Ref="U?"  Part="1"
+AR Path="/5D50DAD7/5D511BC2" Ref="U?"  Part="1"
+AR Path="/5D59955E/5D511BC2" Ref="U?"  Part="1"
+AR Path="/5D6D875D/5D50DAD7/5D511BC2" Ref="U33"  Part="1"
+F 0 "U33" H 5650 5400 50  0000 R CNN
+F 1 "74HC245" H 5650 5300 50  0000 R CNN
+F 2 "Package_SO:SOIC-20W_7.5x12.8mm_P1.27mm" H 5700 4650 50  0001 C CNN
+F 3 "http://www.ti.com/lit/gpn/sn74LS245" H 5700 4650 50  0001 C CNN
+	1    5700 4650
+	-1   0    0    -1
+$EndComp
+Wire Wire Line
+	4700 2900 5200 2900
+Text Label 4950 2900 0    50   ~ 0
+~OE
+Wire Wire Line
+	6200 5150 6500 5150
+Text Label 6500 5150 2    50   ~ 0
+~OE
+$Comp
+L power:GND #PWR?
+U 1 1 5D86A0B0
+P 6300 5450
+AR Path="/5D86A0B0" Ref="#PWR?"  Part="1"
+AR Path="/5D50DAD7/5D86A0B0" Ref="#PWR?"  Part="1"
+AR Path="/5D59955E/5D86A0B0" Ref="#PWR?"  Part="1"
+AR Path="/5D6D875D/5D50DAD7/5D86A0B0" Ref="#PWR0197"  Part="1"
+F 0 "#PWR0197" H 6300 5200 50  0001 C CNN
+F 1 "GND" H 6305 5277 50  0000 C CNN
+F 2 "" H 6300 5450 50  0001 C CNN
+F 3 "" H 6300 5450 50  0001 C CNN
+	1    6300 5450
+	1    0    0    -1
+$EndComp
+Wire Wire Line
+	6300 5450 6300 5050
+Wire Wire Line
+	6300 5050 6200 5050
 $EndSCHEMATC
