File: KiCAD/8-Bit CPU/Control_EEPROM.sch (KiCad schematic (older format))
At the start: 10 parts, among them U36 74HC1G00, U37 74HC1G00, U38 28C64B, U39 74HC245

Commit message: KiCAD files update & Gerbers
Parts:
- renumbered C47 to C44, C46 to C45, C48 to C46, D89 to D93, R39 to R30, R38 to R31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
Connections:
- net ~BE renamed ~CS
