File: KiCAD/8-Bit CPU/Control_ISP.sch (KiCad schematic (older format))
At the start: 14 parts, among them J3 AVRISP, J4 I2C, U34 ATmega16-16AU, U35 CAT24C256

Commit message: KiCAD files update & Gerbers
Parts:
- added R35, R37, R38: 10k, Resistor_SMD:R_0805_2012Metric, symbol Device:R
- renumbered C41 to C47, C42 to C48, C43 to C49, C44 to C50, C45 to C51, D88 to D94, J4 to J3, J3 to J4, R36 to R32, R37 to R33, R35 to R34, R34 to R36, U35 to U42, U34 to U43
Connections:
- net DIR: now also R35.2
- net GND: now also R37.2, R38.2
- net VCC: now also R35.1
- net ~EE: now reaches R36.2, U43.26 (PC7)
- net ~EE: now also R38.1
- net ~OE renamed ~AE
- net ~AE: now also R37.1
Other:
- note added: "Signals Summary:\n\n~AE~: Address Buffer Enable Output\n~EE~: EEPROM Enable Output\n~AS~: EEPROM A Select\n~BS~: EEPROM B Select\n~CS~: EEPROM C Select\nDIR: ~Read~/Write\nWR: Write (Pulse only)"
- moved on the sheet: C47, C48, C49, C50, C51, D94, J3, J4, R32, R33, R34, R36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
