File: KiCAD/8-Bit CPU/Control_InstReg.sch (KiCad schematic (older format))
At the start: 4 parts, among them U33 74HC377

Commit message: KiCAD files update & Gerbers
Parts:
- renumbered C40 to C38, D87 to D91, R33 to R27, U33 to U31
Changed lines of the file:
@@
 Title ""
 Date ""
-Rev ""
+Rev "C"
 Comp ""
 Comment1 ""
@@
 AR Path="/5D57D692/5D582E53" Ref="#PWR?"  Part="1"
 AR Path="/5D506496/5D582E53" Ref="#PWR?"  Part="1"
-AR Path="/5D6D875D/5D506496/5D582E53" Ref="#PWR0202"  Part="1"
-F 0 "#PWR0202" H 5600 2750 50  0001 C CNN
+AR Path="/5D6D875D/5D506496/5D582E53" Ref="#PWR0183"  Part="1"
+F 0 "#PWR0183" H 5600 2750 50  0001 C CNN
 F 1 "VCC" H 5617 3073 50  0000 C CNN
 F 2 "" H 5600 2900 50  0001 C CNN
@@
 AR Path="/5D57D692/5D582C57" Ref="#PWR?"  Part="1"
 AR Path="/5D506496/5D582C57" Ref="#PWR?"  Part="1"
-AR Path="/5D6D875D/5D506496/5D582C57" Ref="#PWR0203"  Part="1"
-F 0 "#PWR0203" H 5600 4400 50  0001 C CNN
+AR Path="/5D6D875D/5D506496/5D582C57" Ref="#PWR0186"  Part="1"
+F 0 "#PWR0186" H 5600 4400 50  0001 C CNN
 F 1 "GND" H 5605 4477 50  0000 C CNN
 F 2 "" H 5600 4650 50  0001 C CNN
@@
 AR Path="/5D57D692/5D581DE8" Ref="#PWR?"  Part="1"
 AR Path="/5D506496/5D581DE8" Ref="#PWR?"  Part="1"
-AR Path="/5D6D875D/5D506496/5D581DE8" Ref="#PWR0204"  Part="1"
-F 0 "#PWR0204" H 6200 4200 50  0001 C CNN
+AR Path="/5D6D875D/5D506496/5D581DE8" Ref="#PWR0185"  Part="1"
+F 0 "#PWR0185" H 6200 4200 50  0001 C CNN
 F 1 "VCC" H 6217 4523 50  0000 C CNN
 F 2 "" H 6200 4350 50  0001 C CNN
@@
 AR Path="/5D57D692/5D581DE2" Ref="#PWR?"  Part="1"
 AR Path="/5D506496/5D581DE2" Ref="#PWR?"  Part="1"
-AR Path="/5D6D875D/5D506496/5D581DE2" Ref="#PWR0205"  Part="1"
-F 0 "#PWR0205" H 6200 4400 50  0001 C CNN
+AR Path="/5D6D875D/5D506496/5D581DE2" Ref="#PWR0187"  Part="1"
+F 0 "#PWR0187" H 6200 4400 50  0001 C CNN
 F 1 "GND" H 6205 4477 50  0000 C CNN
 F 2 "" H 6200 4650 50  0001 C CNN
@@
 AR Path="/5D57D692/5D581DDB" Ref="C?"  Part="1"
 AR Path="/5D506496/5D581DDB" Ref="C?"  Part="1"
-AR Path="/5D6D875D/5D506496/5D581DDB" Ref="C40"  Part="1"
-F 0 "C40" H 6315 4546 50  0000 L CNN
+AR Path="/5D6D875D/5D506496/5D581DDB" Ref="C38"  Part="1"
+F 0 "C38" H 6315 4546 50  0000 L CNN
 F 1 "100n" H 6315 4455 50  0000 L CNN
 F 2 "Capacitor_SMD:C_0805_2012Metric" H 6238 4350 50  0001 C CNN
@@
 $EndComp
 $Comp
-L 74xx:74LS377 U33
+L 74xx:74LS377 U31
 U 1 1 5D57D7D8
 P 5600 3700
-F 0 "U33" H 5650 4500 50  0000 L CNN
+F 0 "U31" H 5650 4500 50  0000 L CNN
 F 1 "74HC377" H 5650 4400 50  0000 L CNN
 F 2 "Package_SO:SOIC-20W_7.5x12.8mm_P1.27mm" H 5600 3700 50  0001 C CNN
@@
 AR Path="/5D57D692/5D5C5628" Ref="#PWR?"  Part="1"
 AR Path="/5D506496/5D5C5628" Ref="#PWR?"  Part="1"
-AR Path="/5D6D875D/5D506496/5D5C5628" Ref="#PWR0201"  Part="1"
-F 0 "#PWR0201" H 4450 3100 50  0001 C CNN
+AR Path="/5D6D875D/5D506496/5D5C5628" Ref="#PWR0184"  Part="1"
+F 0 "#PWR0184" H 4450 3100 50  0001 C CNN
 F 1 "VCC" H 4467 3423 50  0000 C CNN
 F 2 "" H 4450 3250 50  0001 C CNN
@@
 AR Path="/5D4EE537/5D5C4DA9" Ref="R?"  Part="1"
 AR Path="/5D506496/5D5C4DA9" Ref="R?"  Part="1"
-AR Path="/5D6D875D/5D506496/5D5C4DA9" Ref="R33"  Part="1"
-F 0 "R33" H 4350 3850 50  0000 R CNN
+AR Path="/5D6D875D/5D506496/5D5C4DA9" Ref="R27"  Part="1"
+F 0 "R27" H 4350 3850 50  0000 R CNN
 F 1 "1k" H 4350 3950 50  0000 R CNN
 F 2 "Resistor_SMD:R_0805_2012Metric" V 4380 3900 50  0001 C CNN
@@
 AR Path="/5D4EE537/5D5C4DAF" Ref="D?"  Part="1"
 AR Path="/5D506496/5D5C4DAF" Ref="D?"  Part="1"
-AR Path="/5D6D875D/5D506496/5D5C4DAF" Ref="D87"  Part="1"
-F 0 "D87" V 4488 3578 50  0000 L CNN
+AR Path="/5D6D875D/5D506496/5D5C4DAF" Ref="D91"  Part="1"
+F 0 "D91" V 4488 3578 50  0000 L CNN
 F 1 "LED" V 4397 3578 50  0000 L CNN
 F 2 "LED_SMD:LED_0805_2012Metric" H 4450 3500 50  0001 C CNN
