File: KiCAD/8-Bit CPU/Decimal Display.sch (KiCad schematic (older format))
At the start: 11 parts, among them J1 AVRISP, SW6 SW_DIP_x02, U18 ATmega48-20AU, U19 FJ4401AG

Commit message: KiCAD cleanup - Revision A
Revision A Known Issues:
 * ATTiny45 has incorrect footprint
 * Flags register is redundant (The ATMega16's output port is a register)
 * Power jack pinout is wrong (12V shorted to ground)
 * Step counter reset logic is wrong (Active high signalling, Active low input)
 * ALU output indicator not connected
 * HLT indicator missing
 * EEPROMs can't be page written due to addressing setup (minor annoyance)
 * Flags Logic uses NAND gates instead of AND (fixed on the board I built)
 * Programmer needs to be able to toggle EEPROM outputs and Addressing Devices
    with different signals to enable reading.
Other:
- note added: "Using these pins as inputs isn’t the best idea.\nMake PortD Input PortB Output"
Changed lines of the file:
@@
 $Descr A4 11693 8268
 encoding utf-8
-Sheet 12 30
+Sheet 12 29
 Title ""
 Date ""
@@
 Wire Wire Line
 	4900 4200 5300 4200
+Text Notes 5950 2700 0    100  ~ 0
+Using these pins as inputs isn’t the best idea.\nMake PortD Input PortB Output
 Wire Bus Line
 	6000 5100 6000 5800

Commit message: KiCAD files update & Gerbers
Other:
- note removed: "Using these pins as inputs isn’t the best idea.\nMake PortD Input PortB Output"
Changed lines of the file:
@@
 Title ""
 Date ""
-Rev ""
+Rev "C"
 Comp ""
 Comment1 ""
@@
 AR Path="/5D39D95E/5D3E5FC4" Ref="#PWR?"  Part="1"
 AR Path="/5D3E4F90/5D3E5FC4" Ref="#PWR?"  Part="1"
-AR Path="/5D5DCCF9/5D3E5FC4" Ref="#PWR0113"  Part="1"
+AR Path="/5D5DCCF9/5D3E5FC4" Ref="#PWR0112"  Part="1"
 AR Path="/5D5C9807/5D3E5FC4" Ref="#PWR?"  Part="1"
-F 0 "#PWR0113" H 6450 3600 50  0001 C CNN
+F 0 "#PWR0112" H 6450 3600 50  0001 C CNN
 F 1 "GND" H 6455 3677 50  0000 C CNN
 F 2 "" H 6450 3850 50  0001 C CNN
@@
 AR Path="/5D39D95E/5D3E604C" Ref="#PWR?"  Part="1"
 AR Path="/5D3E4F90/5D3E604C" Ref="#PWR?"  Part="1"
-AR Path="/5D5DCCF9/5D3E604C" Ref="#PWR0112"  Part="1"
+AR Path="/5D5DCCF9/5D3E604C" Ref="#PWR0111"  Part="1"
 AR Path="/5D5C9807/5D3E604C" Ref="#PWR?"  Part="1"
-F 0 "#PWR0112" H 6250 3250 50  0001 C CNN
+F 0 "#PWR0111" H 6250 3250 50  0001 C CNN
 F 1 "VCC" V 6250 3500 50  0000 L CNN
 F 2 "" H 6250 3400 50  0001 C CNN
@@
 AR Path="/5D39D95E/5D3E6086" Ref="#PWR?"  Part="1"
 AR Path="/5D3E4F90/5D3E6086" Ref="#PWR?"  Part="1"
-AR Path="/5D5DCCF9/5D3E6086" Ref="#PWR0105"  Part="1"
+AR Path="/5D5DCCF9/5D3E6086" Ref="#PWR0107"  Part="1"
 AR Path="/5D5C9807/5D3E6086" Ref="#PWR?"  Part="1"
-F 0 "#PWR0105" H 1050 800 50  0001 C CNN
+F 0 "#PWR0107" H 1050 800 50  0001 C CNN
 F 1 "GND" H 1055 877 50  0000 C CNN
 F 2 "" H 1050 1050 50  0001 C CNN
@@
 AR Path="/5D39D95E/5D3E60B2" Ref="#PWR?"  Part="1"
 AR Path="/5D3E4F90/5D3E60B2" Ref="#PWR?"  Part="1"
-AR Path="/5D5DCCF9/5D3E60B2" Ref="#PWR0108"  Part="1"
+AR Path="/5D5DCCF9/5D3E60B2" Ref="#PWR0106"  Part="1"
 AR Path="/5D5C9807/5D3E60B2" Ref="#PWR?"  Part="1"
-F 0 "#PWR0108" H 1850 600 50  0001 C CNN
+F 0 "#PWR0106" H 1850 600 50  0001 C CNN
 F 1 "VCC" H 1867 923 50  0000 C CNN
 F 2 "" H 1850 750 50  0001 C CNN
@@
 AR Path="/5D39D95E/5D3E60CD" Ref="#PWR?"  Part="1"
 AR Path="/5D3E4F90/5D3E60CD" Ref="#PWR?"  Part="1"
-AR Path="/5D5DCCF9/5D3E60CD" Ref="#PWR0107"  Part="1"
+AR Path="/5D5DCCF9/5D3E60CD" Ref="#PWR0108"  Part="1"
 AR Path="/5D5C9807/5D3E60CD" Ref="#PWR?"  Part="1"
-F 0 "#PWR0107" H 1450 800 50  0001 C CNN
+F 0 "#PWR0108" H 1450 800 50  0001 C CNN
 F 1 "GND" H 1455 877 50  0000 C CNN
 F 2 "" H 1450 1050 50  0001 C CNN
@@
 AR Path="/5D39D95E/5D3E6173" Ref="#PWR?"  Part="1"
 AR Path="/5D3E4F90/5D3E6173" Ref="#PWR?"  Part="1"
-AR Path="/5D5DCCF9/5D3E6173" Ref="#PWR0106"  Part="1"
+AR Path="/5D5DCCF9/5D3E6173" Ref="#PWR0105"  Part="1"
 AR Path="/5D5C9807/5D3E6173" Ref="#PWR?"  Part="1"
-F 0 "#PWR0106" H 1450 600 50  0001 C CNN
+F 0 "#PWR0105" H 1450 600 50  0001 C CNN
 F 1 "VCC" H 1467 923 50  0000 C CNN
 F 2 "" H 1450 750 50  0001 C CNN
@@
 AR Path="/5D39D95E/5D553D74" Ref="#PWR?"  Part="1"
 AR Path="/5D3E4F90/5D553D74" Ref="#PWR?"  Part="1"
-AR Path="/5D5DCCF9/5D553D74" Ref="#PWR0111"  Part="1"
+AR Path="/5D5DCCF9/5D553D74" Ref="#PWR0115"  Part="1"
 AR Path="/5D5C9807/5D553D74" Ref="#PWR?"  Part="1"
-F 0 "#PWR0111" H 4300 5750 50  0001 C CNN
+F 0 "#PWR0115" H 4300 5750 50  0001 C CNN
 F 1 "GND" H 4305 5827 50  0000 C CNN
 F 2 "" H 4300 6000 50  0001 C CNN
@@
 AR Path="/5D39D95E/5D6838FB" Ref="#PWR?"  Part="1"
 AR Path="/5D3E4F90/5D6838FB" Ref="#PWR?"  Part="1"
-AR Path="/5D5DCCF9/5D6838FB" Ref="#PWR0115"  Part="1"
+AR Path="/5D5DCCF9/5D6838FB" Ref="#PWR0113"  Part="1"
 AR Path="/5D5C9807/5D6838FB" Ref="#PWR?"  Part="1"
-F 0 "#PWR0115" H 7900 3700 50  0001 C CNN
+F 0 "#PWR0113" H 7900 3700 50  0001 C CNN
 F 1 "GND" H 7905 3777 50  0000 C CNN
 F 2 "" H 7900 3950 50  0001 C CNN
@@
 Wire Wire Line
 	4900 4200 5300 4200
-Text Notes 5950 2700 0    100  ~ 0
-Using these pins as inputs isn’t the best idea.\nMake PortD Input PortB Output
 Wire Bus Line
 	6000 5100 6000 5800
