File: KiCAD/8-Bit CPU/LED.sch (KiCad schematic (older format))
At the start: 10 parts

Commit message: KiCAD files update & Gerbers
Parts:
- renumbered D96 to D100, D97 to D101, D98 to D102, D99 to D103, D92 to D96, D93 to D97, D94 to D98, D95 to D99, RN29 to RN31, RN30 to RN32
Changed lines of the file:
@@
 $Descr A4 11693 8268
 encoding utf-8
-Sheet 8 29
+Sheet 15 29
 Title ""
 Date ""
-Rev ""
+Rev "C"
 Comp ""
 Comment1 ""
@@
 AR Path="/5D51F1A5/5D4F3A9B/5D70B41A" Ref="RN?"  Part="1"
 AR Path="/5D5718A3/5D70B41A" Ref="RN?"  Part="1"
-AR Path="/5D6D875D/5D5718A3/5D70B41A" Ref="RN29"  Part="1"
+AR Path="/5D6D875D/5D5718A3/5D70B41A" Ref="RN31"  Part="1"
 AR Path="/5D7088B6/5D408B74/5D70B41A" Ref="RN1"  Part="1"
 AR Path="/5D643828/5D450B31/5D5FFFE8/5D70B41A" Ref="RN13"  Part="1"
 AR Path="/5D643828/5D430931/5D70B41A" Ref="RN3"  Part="1"
-AR Path="/5D613953/5D5AF10D/5D70B41A" Ref="RN21"  Part="1"
-AR Path="/5D613953/5D5E5DC0/5D70B41A" Ref="RN23"  Part="1"
+AR Path="/5D613953/5D5AF10D/5D70B41A" Ref="RN22"  Part="1"
+AR Path="/5D613953/5D5E5DC0/5D70B41A" Ref="RN24"  Part="1"
 AR Path="/5D5EAD14/5D70B41A" Ref="RN?"  Part="1"
-F 0 "RN29" V 5283 2700 50  0000 C CNN
+F 0 "RN31" V 5283 2700 50  0000 C CNN
 F 1 "1k" V 5374 2700 50  0000 C CNN
 F 2 "Resistor_SMD:R_Array_Concave_4x0603" V 5975 2700 50  0001 C CNN
@@
 AR Path="/5D51F1A5/5D4F3A9B/5D70B41B" Ref="D?"  Part="1"
 AR Path="/5D5718A3/5D70B41B" Ref="D?"  Part="1"
-AR Path="/5D6D875D/5D5718A3/5D70B41B" Ref="D92"  Part="1"
+AR Path="/5D6D875D/5D5718A3/5D70B41B" Ref="D96"  Part="1"
 AR Path="/5D7088B6/5D408B74/5D70B41B" Ref="D4"  Part="1"
 AR Path="/5D643828/5D450B31/5D5FFFE8/5D70B41B" Ref="D24"  Part="1"
 AR Path="/5D643828/5D430931/5D70B41B" Ref="D15"  Part="1"
-AR Path="/5D613953/5D5AF10D/5D70B41B" Ref="D48"  Part="1"
-AR Path="/5D613953/5D5E5DC0/5D70B41B" Ref="D56"  Part="1"
+AR Path="/5D613953/5D5AF10D/5D70B41B" Ref="D52"  Part="1"
+AR Path="/5D613953/5D5E5DC0/5D70B41B" Ref="D60"  Part="1"
 AR Path="/5D5EAD14/5D70B41B" Ref="D?"  Part="1"
-F 0 "D92" H 6342 1745 50  0000 C CNN
+F 0 "D96" H 6342 1745 50  0000 C CNN
 F 1 "LED" H 6342 1836 50  0000 C CNN
 F 2 "LED_SMD:LED_0805_2012Metric" H 6350 2000 50  0001 C CNN
@@
 AR Path="/5D51F1A5/5D4F3A9B/5D70B41C" Ref="D?"  Part="1"
 AR Path="/5D5718A3/5D70B41C" Ref="D?"  Part="1"
-AR Path="/5D6D875D/5D5718A3/5D70B41C" Ref="D93"  Part="1"
+AR Path="/5D6D875D/5D5718A3/5D70B41C" Ref="D97"  Part="1"
 AR Path="/5D7088B6/5D408B74/5D70B41C" Ref="D5"  Part="1"
 AR Path="/5D643828/5D450B31/5D5FFFE8/5D70B41C" Ref="D25"  Part="1"
 AR Path="/5D643828/5D430931/5D70B41C" Ref="D16"  Part="1"
-AR Path="/5D613953/5D5AF10D/5D70B41C" Ref="D49"  Part="1"
-AR Path="/5D613953/5D5E5DC0/5D70B41C" Ref="D57"  Part="1"
+AR Path="/5D613953/5D5AF10D/5D70B41C" Ref="D53"  Part="1"
+AR Path="/5D613953/5D5E5DC0/5D70B41C" Ref="D61"  Part="1"
 AR Path="/5D5EAD14/5D70B41C" Ref="D?"  Part="1"
-F 0 "D93" H 6342 2245 50  0000 C CNN
+F 0 "D97" H 6342 2245 50  0000 C CNN
 F 1 "LED" H 6342 2336 50  0000 C CNN
 F 2 "LED_SMD:LED_0805_2012Metric" H 6350 2500 50  0001 C CNN
@@
 AR Path="/5D51F1A5/5D4F3A9B/5D70B41D" Ref="D?"  Part="1"
 AR Path="/5D5718A3/5D70B41D" Ref="D?"  Part="1"
-AR Path="/5D6D875D/5D5718A3/5D70B41D" Ref="D94"  Part="1"
+AR Path="/5D6D875D/5D5718A3/5D70B41D" Ref="D98"  Part="1"
 AR Path="/5D7088B6/5D408B74/5D70B41D" Ref="D6"  Part="1"
 AR Path="/5D643828/5D450B31/5D5FFFE8/5D70B41D" Ref="D26"  Part="1"
 AR Path="/5D643828/5D430931/5D70B41D" Ref="D17"  Part="1"
-AR Path="/5D613953/5D5AF10D/5D70B41D" Ref="D50"  Part="1"
-AR Path="/5D613953/5D5E5DC0/5D70B41D" Ref="D58"  Part="1"
+AR Path="/5D613953/5D5AF10D/5D70B41D" Ref="D54"  Part="1"
+AR Path="/5D613953/5D5E5DC0/5D70B41D" Ref="D62"  Part="1"
 AR Path="/5D5EAD14/5D70B41D" Ref="D?"  Part="1"
-F 0 "D94" H 6342 2745 50  0000 C CNN
+F 0 "D98" H 6342 2745 50  0000 C CNN
 F 1 "LED" H 6342 2836 50  0000 C CNN
 F 2 "LED_SMD:LED_0805_2012Metric" H 6350 3000 50  0001 C CNN
@@
 AR Path="/5D51F1A5/5D4F3A9B/5D70B41E" Ref="D?"  Part="1"
 AR Path="/5D5718A3/5D70B41E" Ref="D?"  Part="1"
-AR Path="/5D6D875D/5D5718A3/5D70B41E" Ref="D95"  Part="1"
+AR Path="/5D6D875D/5D5718A3/5D70B41E" Ref="D99"  Part="1"
 AR Path="/5D7088B6/5D408B74/5D70B41E" Ref="D7"  Part="1"
 AR Path="/5D643828/5D450B31/5D5FFFE8/5D70B41E" Ref="D27"  Part="1"
 AR Path="/5D643828/5D430931/5D70B41E" Ref="D18"  Part="1"
-AR Path="/5D613953/5D5AF10D/5D70B41E" Ref="D51"  Part="1"
-AR Path="/5D613953/5D5E5DC0/5D70B41E" Ref="D59"  Part="1"
+AR Path="/5D613953/5D5AF10D/5D70B41E" Ref="D55"  Part="1"
+AR Path="/5D613953/5D5E5DC0/5D70B41E" Ref="D63"  Part="1"
 AR Path="/5D5EAD14/5D70B41E" Ref="D?"  Part="1"
-F 0 "D95" H 6342 3245 50  0000 C CNN
+F 0 "D99" H 6342 3245 50  0000 C CNN
 F 1 "LED" H 6342 3336 50  0000 C CNN
 F 2 "LED_SMD:LED_0805_2012Metric" H 6350 3500 50  0001 C CNN
@@
 AR Path="/5D51F1A5/5D4F3A9B/5D70B41F" Ref="RN?"  Part="1"
 AR Path="/5D5718A3/5D70B41F" Ref="RN?"  Part="1"
-AR Path="/5D6D875D/5D5718A3/5D70B41F" Ref="RN30"  Part="1"
+AR Path="/5D6D875D/5D5718A3/5D70B41F" Ref="RN32"  Part="1"
 AR Path="/5D7088B6/5D408B74/5D70B41F" Ref="RN2"  Part="1"
 AR Path="/5D643828/5D450B31/5D5FFFE8/5D70B41F" Ref="RN14"  Part="1"
 AR Path="/5D643828/5D430931/5D70B41F" Ref="RN4"  Part="1"
-AR Path="/5D613953/5D5AF10D/5D70B41F" Ref="RN22"  Part="1"
-AR Path="/5D613953/5D5E5DC0/5D70B41F" Ref="RN24"  Part="1"
+AR Path="/5D613953/5D5AF10D/5D70B41F" Ref="RN23"  Part="1"
+AR Path="/5D613953/5D5E5DC0/5D70B41F" Ref="RN25"  Part="1"
 AR Path="/5D5EAD14/5D70B41F" Ref="RN?"  Part="1"
-F 0 "RN30" V 5283 4700 50  0000 C CNN
+F 0 "RN32" V 5283 4700 50  0000 C CNN
 F 1 "1k" V 5374 4700 50  0000 C CNN
 F 2 "Resistor_SMD:R_Array_Concave_4x0603" V 5975 4700 50  0001 C CNN
@@
 AR Path="/5D51F1A5/5D4F3A9B/5D70B420" Ref="D?"  Part="1"
 AR Path="/5D5718A3/5D70B420" Ref="D?"  Part="1"
-AR Path="/5D6D875D/5D5718A3/5D70B420" Ref="D96"  Part="1"
+AR Path="/5D6D875D/5D5718A3/5D70B420" Ref="D100"  Part="1"
 AR Path="/5D7088B6/5D408B74/5D70B420" Ref="D8"  Part="1"
 AR Path="/5D643828/5D450B31/5D5FFFE8/5D70B420" Ref="D28"  Part="1"
 AR Path="/5D643828/5D430931/5D70B420" Ref="D19"  Part="1"
-AR Path="/5D613953/5D5AF10D/5D70B420" Ref="D52"  Part="1"
-AR Path="/5D613953/5D5E5DC0/5D70B420" Ref="D60"  Part="1"
+AR Path="/5D613953/5D5AF10D/5D70B420" Ref="D56"  Part="1"
+AR Path="/5D613953/5D5E5DC0/5D70B420" Ref="D64"  Part="1"
 AR Path="/5D5EAD14/5D70B420" Ref="D?"  Part="1"
-F 0 "D96" H 6342 3745 50  0000 C CNN
+F 0 "D100" H 6342 3745 50  0000 C CNN
 F 1 "LED" H 6342 3836 50  0000 C CNN
 F 2 "LED_SMD:LED_0805_2012Metric" H 6350 4000 50  0001 C CNN
@@
 AR Path="/5D51F1A5/5D4F3A9B/5D70B421" Ref="D?"  Part="1"
 AR Path="/5D5718A3/5D70B421" Ref="D?"  Part="1"
-AR Path="/5D6D875D/5D5718A3/5D70B421" Ref="D97"  Part="1"
+AR Path="/5D6D875D/5D5718A3/5D70B421" Ref="D101"  Part="1"
 AR Path="/5D7088B6/5D408B74/5D70B421" Ref="D9"  Part="1"
 AR Path="/5D643828/5D450B31/5D5FFFE8/5D70B421" Ref="D29"  Part="1"
 AR Path="/5D643828/5D430931/5D70B421" Ref="D20"  Part="1"
-AR Path="/5D613953/5D5AF10D/5D70B421" Ref="D53"  Part="1"
-AR Path="/5D613953/5D5E5DC0/5D70B421" Ref="D61"  Part="1"
+AR Path="/5D613953/5D5AF10D/5D70B421" Ref="D57"  Part="1"
+AR Path="/5D613953/5D5E5DC0/5D70B421" Ref="D65"  Part="1"
 AR Path="/5D5EAD14/5D70B421" Ref="D?"  Part="1"
-F 0 "D97" H 6342 4245 50  0000 C CNN
+F 0 "D101" H 6342 4245 50  0000 C CNN
 F 1 "LED" H 6342 4336 50  0000 C CNN
 F 2 "LED_SMD:LED_0805_2012Metric" H 6350 4500 50  0001 C CNN
@@
 AR Path="/5D51F1A5/5D4F3A9B/5D70B422" Ref="D?"  Part="1"
 AR Path="/5D5718A3/5D70B422" Ref="D?"  Part="1"
-AR Path="/5D6D875D/5D5718A3/5D70B422" Ref="D98"  Part="1"
+AR Path="/5D6D875D/5D5718A3/5D70B422" Ref="D102"  Part="1"
 AR Path="/5D7088B6/5D408B74/5D70B422" Ref="D10"  Part="1"
 AR Path="/5D643828/5D450B31/5D5FFFE8/5D70B422" Ref="D30"  Part="1"
 AR Path="/5D643828/5D430931/5D70B422" Ref="D21"  Part="1"
-AR Path="/5D613953/5D5AF10D/5D70B422" Ref="D54"  Part="1"
-AR Path="/5D613953/5D5E5DC0/5D70B422" Ref="D62"  Part="1"
+AR Path="/5D613953/5D5AF10D/5D70B422" Ref="D58"  Part="1"
+AR Path="/5D613953/5D5E5DC0/5D70B422" Ref="D66"  Part="1"
 AR Path="/5D5EAD14/5D70B422" Ref="D?"  Part="1"
-F 0 "D98" H 6342 4745 50  0000 C CNN
+F 0 "D102" H 6342 4745 50  0000 C CNN
 F 1 "LED" H 6342 4836 50  0000 C CNN
 F 2 "LED_SMD:LED_0805_2012Metric" H 6350 5000 50  0001 C CNN
@@
 AR Path="/5D51F1A5/5D4F3A9B/5D70B423" Ref="D?"  Part="1"
 AR Path="/5D5718A3/5D70B423" Ref="D?"  Part="1"
-AR Path="/5D6D875D/5D5718A3/5D70B423" Ref="D99"  Part="1"
+AR Path="/5D6D875D/5D5718A3/5D70B423" Ref="D103"  Part="1"
 AR Path="/5D7088B6/5D408B74/5D70B423" Ref="D11"  Part="1"
 AR Path="/5D643828/5D450B31/5D5FFFE8/5D70B423" Ref="D31"  Part="1"
 AR Path="/5D643828/5D430931/5D70B423" Ref="D22"  Part="1"
-AR Path="/5D613953/5D5AF10D/5D70B423" Ref="D55"  Part="1"
-AR Path="/5D613953/5D5E5DC0/5D70B423" Ref="D63"  Part="1"
+AR Path="/5D613953/5D5AF10D/5D70B423" Ref="D59"  Part="1"
+AR Path="/5D613953/5D5E5DC0/5D70B423" Ref="D67"  Part="1"
 AR Path="/5D5EAD14/5D70B423" Ref="D?"  Part="1"
-F 0 "D99" H 6342 5245 50  0000 C CNN
+F 0 "D103" H 6342 5245 50  0000 C CNN
 F 1 "LED" H 6342 5336 50  0000 C CNN
 F 2 "LED_SMD:LED_0805_2012Metric" H 6350 5500 50  0001 C CNN
@@
 AR Path="/5D51F1A5/5D4F3A9B/5D4F513A" Ref="#PWR?"  Part="1"
 AR Path="/5D5718A3/5D4F513A" Ref="#PWR?"  Part="1"
-AR Path="/5D6D875D/5D5718A3/5D4F513A" Ref="#PWR0267"  Part="1"
+AR Path="/5D6D875D/5D5718A3/5D4F513A" Ref="#PWR0263"  Part="1"
 AR Path="/5D7088B6/5D408B74/5D4F513A" Ref="#PWR019"  Part="1"
 AR Path="/5D643828/5D450B31/5D5FFFE8/5D4F513A" Ref="#PWR066"  Part="1"
 AR Path="/5D643828/5D430931/5D4F513A" Ref="#PWR031"  Part="1"
-AR Path="/5D613953/5D5AF10D/5D4F513A" Ref="#PWR0145"  Part="1"
-AR Path="/5D613953/5D5E5DC0/5D4F513A" Ref="#PWR0146"  Part="1"
+AR Path="/5D613953/5D5AF10D/5D4F513A" Ref="#PWR0141"  Part="1"
+AR Path="/5D613953/5D5E5DC0/5D4F513A" Ref="#PWR0142"  Part="1"
 AR Path="/5D5EAD14/5D4F513A" Ref="#PWR?"  Part="1"
-F 0 "#PWR0267" H 6800 5550 50  0001 C CNN
+F 0 "#PWR0263" H 6800 5550 50  0001 C CNN
 F 1 "GND" H 6805 5627 50  0000 C CNN
 F 2 "" H 6800 5800 50  0001 C CNN
