File: KiCAD/8-Bit CPU/ProgCount.sch (KiCad schematic (older format))
At the start: 12 parts, among them U1 74HC161, U2 74HC161, U3 74HC245

Commit message: KiCAD files update & Gerbers
Parts:
- renumbered C3 to C2, C2 to C3, D3 to D2, D2 to D3, R4 to R3, R3 to R4, U3 to U2, U2 to U3
Connections:
- net EN: no longer U1.10 (CET)
- net VCC: now also U1.10 (CET)
Changed lines of the file:
@@
 encoding utf-8
 Sheet 2 29
-Title ""
+Title "Program Counter"
 Date ""
-Rev ""
+Rev "C"
 Comp ""
 Comment1 ""
@@
 $EndDescr
 $Comp
-L power:GND #PWR012
+L power:GND #PWR018
 U 1 1 5D3F5EDC
 P 5800 5400
-F 0 "#PWR012" H 5800 5150 50  0001 C CNN
+F 0 "#PWR018" H 5800 5150 50  0001 C CNN
 F 1 "GND" H 5900 5300 50  0000 C CNN
 F 2 "" H 5800 5400 50  0001 C CNN
@@
 $EndComp
 $Comp
-L power:GND #PWR08
+L power:GND #PWR012
 U 1 1 5D3F5EE2
 P 4050 4300
-F 0 "#PWR08" H 4050 4050 50  0001 C CNN
+F 0 "#PWR012" H 4050 4050 50  0001 C CNN
 F 1 "GND" H 4150 4200 50  0000 C CNN
 F 2 "" H 4050 4300 50  0001 C CNN
@@
 $EndComp
 $Comp
-L power:GND #PWR017
+L power:GND #PWR014
 U 1 1 5D3F5F1F
 P 9100 4300
-F 0 "#PWR017" H 9100 4050 50  0001 C CNN
+F 0 "#PWR014" H 9100 4050 50  0001 C CNN
 F 1 "GND" H 9200 4200 50  0000 C CNN
 F 2 "" H 9100 4300 50  0001 C CNN
@@
 $EndComp
 $Comp
-L Device:C C3
+L Device:C C2
 U 1 1 5D3F5F25
 P 9100 4150
-F 0 "C3" H 9215 4196 50  0000 L CNN
+F 0 "C2" H 9215 4196 50  0000 L CNN
 F 1 "100n" H 9215 4105 50  0000 L CNN
 F 2 "Capacitor_SMD:C_0805_2012Metric" H 9138 4000 50  0001 C CNN
@@
 $EndComp
 $Comp
-L Device:C C2
+L Device:C C3
 U 1 1 5D3F5F33
 P 5800 5250
-F 0 "C2" H 5915 5296 50  0000 L CNN
+F 0 "C3" H 5915 5296 50  0000 L CNN
 F 1 "100n" H 5915 5205 50  0000 L CNN
 F 2 "Capacitor_SMD:C_0805_2012Metric" H 5838 5100 50  0001 C CNN
@@
 	2900 3000 3100 3000
 Wire Wire Line
-	2700 3800 3100 3800
-Wire Wire Line
-	2700 4900 2700 3800
-Wire Wire Line
-	4800 4900 2700 4900
-Wire Wire Line
-	3000 3600 2800 3600
-Wire Wire Line
-	3000 3700 3000 3600
-Wire Wire Line
-	3100 3700 3000 3700
-Wire Wire Line
-	2800 4700 4800 4700
-Wire Wire Line
-	2800 3600 2800 4700
-Connection ~ 3000 3600
-Wire Wire Line
-	3100 3600 3000 3600
-Wire Wire Line
-	2900 3500 3100 3500
-Wire Wire Line
-	2900 4600 2900 3500
-Wire Wire Line
-	4800 4600 2900 4600
+	2600 3800 3100 3800
+Wire Wire Line
+	2600 4900 2600 3800
+Wire Wire Line
+	4800 4900 2600 4900
+Wire Wire Line
+	2700 4700 4800 4700
+Wire Wire Line
+	2700 3600 2700 4700
+Wire Wire Line
+	2800 3500 3100 3500
+Wire Wire Line
+	2800 4600 2800 3500
+Wire Wire Line
+	4800 4600 2800 4600
 Wire Wire Line
 	3000 5100 4800 5100
@@
 	9000 3300 9200 3300
 $Comp
-L power:GND #PWR015
+L power:GND #PWR013
 U 1 1 5D3F602F
 P 8500 4300
-F 0 "#PWR015" H 8500 4050 50  0001 C CNN
+F 0 "#PWR013" H 8500 4050 50  0001 C CNN
 F 1 "GND" H 8600 4200 50  0000 C CNN
 F 2 "" H 8500 4300 50  0001 C CNN
@@
 BUS0
 $Comp
-L power:GND #PWR010
+L power:GND #PWR017
 U 1 1 5D3F605A
 P 5300 5400
-F 0 "#PWR010" H 5300 5150 50  0001 C CNN
+F 0 "#PWR017" H 5300 5150 50  0001 C CNN
 F 1 "GND" H 5400 5300 50  0000 C CNN
 F 2 "" H 5300 5400 50  0001 C CNN
@@
 $EndComp
 $Comp
-L 74xx:74LS161 U2
+L 74xx:74LS161 U3
 U 1 1 5D3F6060
 P 5300 4600
-F 0 "U2" H 5050 5250 50  0000 C CNN
+F 0 "U3" H 5050 5250 50  0000 C CNN
 F 1 "74HC161" H 5500 5250 50  0000 C CNN
 F 2 "Package_SO:SOIC-16_3.9x9.9mm_P1.27mm" H 5300 4600 50  0001 C CNN
@@
 $EndComp
 $Comp
-L power:GND #PWR06
+L power:GND #PWR011
 U 1 1 5D3F6067
 P 3600 4300
-F 0 "#PWR06" H 3600 4050 50  0001 C CNN
+F 0 "#PWR011" H 3600 4050 50  0001 C CNN
 F 1 "GND" H 3700 4200 50  0000 C CNN
 F 2 "" H 3600 4300 50  0001 C CNN
@@
 $EndComp
 $Comp
-L 74xx:74HC245 U3
+L 74xx:74HC245 U2
 U 1 1 5D3F606D
 P 8500 3500
-F 0 "U3" H 8250 4150 50  0000 C CNN
+F 0 "U2" H 8250 4150 50  0000 C CNN
 F 1 "74HC245" H 8700 4150 50  0000 C CNN
 F 2 "jcf:SOIC-20W_7.5x12.8mm_P1.27mm_Rounded" H 8500 3500 50  0001 C CNN
@@
 $EndComp
 $Comp
-L power:VCC #PWR013
+L power:VCC #PWR08
 U 1 1 5D40E16A
 P 8000 3900
-F 0 "#PWR013" H 8000 3750 50  0001 C CNN
+F 0 "#PWR08" H 8000 3750 50  0001 C CNN
 F 1 "VCC" V 8018 4027 50  0000 L CNN
 F 2 "" H 8000 3900 50  0001 C CNN
@@
 CLK
 Wire Wire Line
-	2400 3800 2700 3800
-Connection ~ 2700 3800
+	2400 3800 2600 3800
+Connection ~ 2600 3800
 Text HLabel 1700 3600 0    50   Input ~ 0
 EN
 Wire Wire Line
 	1700 3600 1800 3600
-Connection ~ 2800 3600
+Connection ~ 2700 3600
 Text HLabel 1700 3500 0    50   Input ~ 0
 ~IN
 Wire Wire Line
 	1700 3500 1800 3500
-Connection ~ 2900 3500
-$Comp
-L power:VCC #PWR07
+Connection ~ 2800 3500
+$Comp
+L power:VCC #PWR09
 U 1 1 5D4419F0
 P 4050 4000
-F 0 "#PWR07" H 4050 3850 50  0001 C CNN
+F 0 "#PWR09" H 4050 3850 50  0001 C CNN
 F 1 "VCC" H 4067 4173 50  0000 C CNN
 F 2 "" H 4050 4000 50  0001 C CNN
@@
 $EndComp
 $Comp
-L power:VCC #PWR011
+L power:VCC #PWR016
 U 1 1 5D441C07
 P 5800 5100
-F 0 "#PWR011" H 5800 4950 50  0001 C CNN
+F 0 "#PWR016" H 5800 4950 50  0001 C CNN
 F 1 "VCC" H 5817 5273 50  0000 C CNN
 F 2 "" H 5800 5100 50  0001 C CNN
@@
 	2400 3300 2700 3300
 $Comp
-L power:VCC #PWR05
+L power:VCC #PWR04
 U 1 1 5D4882C7
 P 3600 2700
-F 0 "#PWR05" H 3600 2550 50  0001 C CNN
+F 0 "#PWR04" H 3600 2550 50  0001 C CNN
 F 1 "VCC" H 3617 2873 50  0000 C CNN
 F 2 "" H 3600 2700 50  0001 C CNN
@@
 $EndComp
 $Comp
-L power:VCC #PWR09
+L power:VCC #PWR07
 U 1 1 5D488367
 P 5300 3800
-F 0 "#PWR09" H 5300 3650 50  0001 C CNN
+F 0 "#PWR07" H 5300 3650 50  0001 C CNN
 F 1 "VCC" H 5317 3973 50  0000 C CNN
 F 2 "" H 5300 3800 50  0001 C CNN
@@
 $EndComp
 $Comp
-L power:VCC #PWR014
+L power:VCC #PWR05
 U 1 1 5D488407
 P 8500 2700
-F 0 "#PWR014" H 8500 2550 50  0001 C CNN
+F 0 "#PWR05" H 8500 2550 50  0001 C CNN
 F 1 "VCC" H 8517 2873 50  0000 C CNN
 F 2 "" H 8500 2700 50  0001 C CNN
@@
 $EndComp
 $Comp
-L power:VCC #PWR016
+L power:VCC #PWR010
 U 1 1 5D3E2497
 P 9100 4000
-F 0 "#PWR016" H 9100 3850 50  0001 C CNN
+F 0 "#PWR010" H 9100 3850 50  0001 C CNN
 F 1 "VCC" H 9117 4173 50  0000 C CNN
 F 2 "" H 9100 4000 50  0001 C CNN
@@
 Connection ~ 1800 3500
 Wire Wire Line
-	1800 3500 2900 3500
+	1800 3500 2800 3500
 Wire Wire Line
 	9600 3950 9600 4050
@@
 AR Path="/5D506496/5D5A7363" Ref="#PWR?"  Part="1"
 AR Path="/5D6D875D/5D506496/5D5A7363" Ref="#PWR?"  Part="1"
-AR Path="/5D7088B6/5D5A7363" Ref="#PWR018"  Part="1"
-F 0 "#PWR018" H 9600 3400 50  0001 C CNN
+AR Path="/5D7088B6/5D5A7363" Ref="#PWR06"  Part="1"
+F 0 "#PWR06" H 9600 3400 50  0001 C CNN
 F 1 "VCC" H 9617 3723 50  0000 C CNN
 F 2 "" H 9600 3550 50  0001 C CNN
@@
 AR Path="/5D506496/5D5A736A" Ref="R?"  Part="1"
 AR Path="/5D6D875D/5D506496/5D5A736A" Ref="R?"  Part="1"
-AR Path="/5D7088B6/5D5A736A" Ref="R4"  Part="1"
-F 0 "R4" H 9500 4150 50  0000 R CNN
+AR Path="/5D7088B6/5D5A736A" Ref="R3"  Part="1"
+F 0 "R3" H 9500 4150 50  0000 R CNN
 F 1 "1k" H 9500 4250 50  0000 R CNN
 F 2 "Resistor_SMD:R_0805_2012Metric" V 9530 4200 50  0001 C CNN
@@
 AR Path="/5D506496/5D5A7370" Ref="D?"  Part="1"
 AR Path="/5D6D875D/5D506496/5D5A7370" Ref="D?"  Part="1"
-AR Path="/5D7088B6/5D5A7370" Ref="D3"  Part="1"
-F 0 "D3" V 9638 3878 50  0000 L CNN
+AR Path="/5D7088B6/5D5A7370" Ref="D2"  Part="1"
+F 0 "D2" V 9638 3878 50  0000 L CNN
 F 1 "LED" V 9547 3878 50  0000 L CNN
 F 2 "LED_SMD:LED_0805_2012Metric" H 9600 3800 50  0001 C CNN
@@
 AR Path="/5D506496/5D5B014A" Ref="R?"  Part="1"
 AR Path="/5D6D875D/5D506496/5D5B014A" Ref="R?"  Part="1"
-AR Path="/5D7088B6/5D5B014A" Ref="R3"  Part="1"
-F 0 "R3" H 1700 4250 50  0000 R CNN
+AR Path="/5D7088B6/5D5B014A" Ref="R4"  Part="1"
+F 0 "R4" H 1700 4250 50  0000 R CNN
 F 1 "1k" H 1700 4350 50  0000 R CNN
 F 2 "Resistor_SMD:R_0805_2012Metric" V 1730 4300 50  0001 C CNN
@@
 AR Path="/5D506496/5D5B0150" Ref="D?"  Part="1"
 AR Path="/5D6D875D/5D506496/5D5B0150" Ref="D?"  Part="1"
-AR Path="/5D7088B6/5D5B0150" Ref="D2"  Part="1"
-F 0 "D2" V 1838 3978 50  0000 L CNN
+AR Path="/5D7088B6/5D5B0150" Ref="D3"  Part="1"
+F 0 "D3" V 1838 3978 50  0000 L CNN
 F 1 "LED" V 1747 3978 50  0000 L CNN
 F 2 "LED_SMD:LED_0805_2012Metric" H 1800 3900 50  0001 C CNN
@@
 $EndComp
 $Comp
-L power:GND #PWR04
+L power:GND #PWR015
 U 1 1 5D5B72B4
 P 1800 4600
-F 0 "#PWR04" H 1800 4350 50  0001 C CNN
+F 0 "#PWR015" H 1800 4350 50  0001 C CNN
 F 1 "GND" H 1900 4500 50  0000 C CNN
 F 2 "" H 1800 4600 50  0001 C CNN
@@
 Connection ~ 1800 3600
 Wire Wire Line
-	1800 3600 2800 3600
+	1800 3600 2700 3600
 $Sheet
 S 8200 4700 600  900
@@
 	2400 5100 3000 5100
 Connection ~ 3000 5100
+Wire Wire Line
+	2700 3600 3100 3600
+$Comp
+L power:VCC #PWR?
+U 1 1 5D85779E
+P 3100 3700
+F 0 "#PWR?" H 3100 3550 50  0001 C CNN
+F 1 "VCC" V 3117 3873 50  0000 C CNN
+F 2 "" H 3100 3700 50  0001 C CNN
+F 3 "" H 3100 3700 50  0001 C CNN
+	1    3100 3700
+	0    -1   -1   0
+$EndComp
 Wire Bus Line
 	2800 2400 9300 2400
