File: KiCAD/8-Bit CPU/RAM_Logic.sch (KiCad schematic (older format))
At the start: 18 parts, among them SW4 SW_Push, SW5 SW_Push, U12 74HC00, U13 74HC132

Commit message: KiCAD files update & Gerbers
Parts:
- renumbered C16 to C12, C15 to C13, C12 to C14, C13 to C15, C14 to C16, R14 to R10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
