File: KiCAD/8-Bit CPU/Register.sch (KiCad schematic (older format))
At the start: 18 parts, among them U26 74HC377, U27 74HC245

Commit message: KiCAD files update & Gerbers
Parts:
- renumbered C33 to C32, C34 to C33, D76 to D78, D77 to D79, D78 to D80, D79 to D81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
